Commit message: Fix: try canopenLib changes - update EDS, configs, and launch files

File: crane/tower_crane_moveit_config/config/tower_crane.ros2_control.xacro (robot description, xacro)
@@ -2,5 +2,5 @@
 <robot xmlns:xacro="http://www.ros.org/wiki/xacro">
     <xacro:macro name="tower_crane_ros2_control" params="name initial_positions_file">
-        <xacro:property name="initial_positions" value="${load_yaml(initial_positions_file)['initial_positions']}"/>
+        <xacro:property name="initial_positions" value="${xacro.load_yaml(initial_positions_file)['initial_positions']}"/>
         <ros2_control name="${name}" type="system">
             <hardware>

File: crane/tower_crane_moveit_config/config/tower_crane.urdf.xacro (robot description, xacro)
@@ -2,7 +2,6 @@
 <robot xmlns:xacro="http://www.ros.org/wiki/xacro" name="tower_crane">
     <xacro:arg name="initial_positions_file" default="initial_positions.yaml" />
-    <!-- Import tower_crane URDF file -->
-    <!-- Note: xacro supports $(find package_name) via its own 'find' substitution command. -->
-    <xacro:include filename="$(find tower_crane)/urdf/Tower_crane.urdf" />
+    <!-- Import tower_crane base URDF file (geometry only, no ros2_control) -->
+    <xacro:include filename="$(find tower_crane)/urdf/Tower_crane_base.urdf" />
     <!-- Import control_xacro -->
     <xacro:include filename="tower_crane.ros2_control.xacro" />
