Commit message: working on the moveit part

File: crane/tower_crane/urdf/Tower_crane_base.urdf (robot description, URDF)
Before this commit: robot tower_crane, 6 links, 5 joints
Joints:
- joint hook_joint: limit lower=0 upper=2 effort=50 velocity=0.5 -> lower=0 upper=2 effort=50 velocity=1.0
- joint trolley_joint: limit lower=-2 upper=0.5 effort=20 velocity=0.5 -> lower=-2 upper=0.5 effort=20 velocity=1.0

File: crane/tower_crane_moveit_config/config/tower_crane.urdf.xacro (robot description, xacro)
@@ -3,7 +3,216 @@
     <xacro:arg name="initial_positions_file" default="initial_positions.yaml" />
     <!-- Import tower_crane base URDF file (geometry only, no ros2_control) -->
-    <xacro:include filename="$(find tower_crane)/urdf/Tower_crane_base.urdf" />
-    <!-- Import control_xacro -->
-    <xacro:include filename="tower_crane.ros2_control.xacro" />
-    <xacro:tower_crane_ros2_control name="FakeSystem" initial_positions_file="$(arg initial_positions_file)"/>
+    <link name="world"/>
+    <joint name="world_to_base" type="fixed">
+      <parent link="world"/>
+      <child link="base_base_link"/>
+      <origin rpy="0 0 0" xyz="0 0 0"/>
+    </joint>
+    <link name="base_base_link">
+      <visual>
+        <geometry>
+          <box size="0.45 0.45 0.2"/>
+        </geometry>
+        <material name="">
+          <color rgba="0.79216 0.81961 0.93333 1"/>
+        </material>
+      </visual>
+    </link>
+    <joint name="base_to_base" type="fixed">
+      <parent link="base_base_link"/>
+      <child link="base_link"/>
+      <origin xyz="0 0 2" rpy="0 0 0"/>
+    </joint>
+    <link name="base_link">
+      <inertial>
+        <origin xyz="-0.00054365 0.0005699 -0.90918" rpy="0 0 0" />
+        <mass value="24.622" />
+        <inertia
+          ixx="12.76" ixy="0" ixz="0.01"
+          iyy="12.75" iyz="-0.04" izz="0.70" />
+      </inertial>
+      <visual>
+        <origin xyz="0 0 0" rpy="0 0 0" />
+        <geometry>
+          <mesh  filename="package://tower_crane/meshes/base_link.STL" />
+        </geometry>
+        <material name="">
+          <color rgba="0.79216 0.81961 0.93333 1" />
+        </material>
+      </visual>
+      <collision>
+        <origin  xyz="0 0 0"  rpy="0 0 0" />
+        <geometry>
+          <mesh  filename="package://tower_crane/meshes/base_link.STL" />
+        </geometry>
+      </collision>
+    </link>
+    <joint name="slewing_joint"  type="revolute">
+      <origin xyz="0 0 0.007"  rpy="0 0 0" />
+      <parent  link="base_link" />
+      <child  link="slewing_Link" />
+      <axis  xyz="0 0 1" />
+      <limit  lower="-3.14"  upper="3.14"  effort="100"  velocity="0" />
+    </joint>
+    <link  name="slewing_Link">
+      <inertial>
+        <origin  xyz="-0.000744911036835383 -0.0874649854532076 0.14613338637878"  rpy="0 0 0" />
+        <mass  value="38.2285461245108" />
+        <inertia  ixx=" 32.67"  ixy="0.03" ixz="0.00" iyy="2.25" iyz="2.79" izz=" 31.30" />
+      </inertial>
+      <visual>
+        <origin xyz="0 0 0" rpy="0 0 0" />
+        <geometry>
+          <mesh  filename="package://tower_crane/meshes/slewing_Link.STL" />
+        </geometry>
+        <material  name="">
+          <color  rgba="0.792156862745098 0.819607843137255 0.933333333333333 1" />
+        </material>
+      </visual>
+      <collision>
+        <origin  xyz="0 0 0"  rpy="0 0 0" />
+        <geometry>
+          <mesh  filename="package://tower_crane/meshes/slewing_Link.STL" />
+        </geometry>
+      </collision>
+    </link>
+    <joint  name="trolley_joint"  type="prismatic">
+      <origin  xyz="0.00031802 -1.4078 0.1438"  rpy="0 0 -3.1416" />
+      <parent  link="slewing_Link" />
+      <child  link="trolley_Link" />
+      <axis  xyz="0 1 0" />
+      <limit  lower="-2" upper="0.5" effort="20" velocity="1.0" />
+    </joint>
+    <link  name="trolley_Link">
+      <inertial>
+          <origin  xyz="-0.00252711686986329 -6.66133814775094E-16 -0.146022586184743"  rpy="0 0 0" />
+          <mass  value="0.567964273921575" />
+          <inertia ixx="0.12" ixy="0.00" ixz="0.00"
+                  iyy="0.13" iyz="0.00" izz="0.01" />
+      </inertial>
+      <visual>
+        <origin xyz="0 0 0" rpy="0 0 0" />
+        <geometry>
+          <mesh  filename="package://tower_crane/meshes/trolley_Link.STL" />
+        </geometry>
+        <material  name="">
+          <color  rgba="0.792156862745098 0.819607843137255 0.933333333333333 1" />
+        </material>
+      </visual>
+      <collision>
+        <origin xyz="0 0 0" rpy="0 0 0" />
+        <geometry>
+          <mesh  filename="package://tower_crane/meshes/trolley_Link.STL" />
+        </geometry>
+      </collision>
+    </link>
+    <joint  name="hook_joint" type="prismatic">
+      <origin xyz="-0.013982 0 -1.9126" rpy="0 0 3.1416" />
+      <parent  link="trolley_Link" />
+      <child  link="hook_Link" />
+      <axis  xyz="0 0 1" />
+      <limit  lower="0" upper="2" effort="50" velocity="1.0" />
+    </joint>
+    <link name="hook_Link">
+      <inertial>
+        <origin xyz="0 2.22044604925031E-16 0" rpy="0 0 0" />
+        <mass value="5.0" />
+        <inertia ixx="0.01" ixy="0.00" ixz="0.00"
+                  iyy="0.01" iyz="0.00" izz="0.01" />
+      </inertial>
+      <visual>
+        <origin xyz="0 0 0" rpy="0 0 0" />
+        <geometry>
+          <mesh filename="package://tower_crane/meshes/hook_Link.STL" />
+        </geometry>
+        <material  name="">
+          <color
+            rgba="0.792156862745098 0.819607843137255 0.933333333333333 1" />
+        </material>
+      </visual>
+      <collision>
+        <origin xyz="0 0 0" rpy="0 0 0" />
+        <geometry>
+          <mesh  filename="package://tower_crane/meshes/hook_Link.STL" />
+        </geometry>
+      </collision>
+    </link>
+    <transmission name="slewing_transmission">
+      <type>transmission_interface/SimpleTransmission</type>
+      <joint name="slewing_joint">
+        <hardwareInterface>hardware_interface/PositionJointInterface</hardwareInterface>
+      </joint>
+      <actuator name="slewing_motor">
+        <hardwareInterface>hardware_interface/PositionJointInterface</hardwareInterface>
+        <mechanicalReduction>140.0</mechanicalReduction>
+      </actuator>
+    </transmission>
+    <transmission name="trolley_transmission">
+      <type>transmission_interface/SimpleTransmission</type>
+      <joint name="trolley_joint">
+        <hardwareInterface>hardware_interface/PositionJointInterface</hardwareInterface>
+      </joint>
+      <actuator name="trolley_motor">
+        <hardwareInterface>hardware_interface/PositionJointInterface</hardwareInterface>
+        <mechanicalReduction>10.0</mechanicalReduction>
+      </actuator>
+    </transmission>
+    <transmission name="hoist_transmission">
+      <type>transmission_interface/SimpleTransmission</type>
+      <joint name="hook_joint">
+        <hardwareInterface>hardware_interface/PositionJointInterface</hardwareInterface>
+      </joint>
+      <actuator name="hoist_motor">
+        <hardwareInterface>hardware_interface/PositionJointInterface</hardwareInterface>
+        <mechanicalReduction>40.0</mechanicalReduction>
+      </actuator>
+    </transmission>
+    <xacro:macro name="tower_crane_ros2_control" params="name initial_positions_file">
+      <xacro:property name="initial_positions" value="${xacro.load_yaml(initial_positions_file)['initial_positions']}"/>
+      <ros2_control name="${name}" type="system">
+        <hardware>
+            <plugin>ros2_control_demo_hardware/RRBotSystemPositionOnlyHardware</plugin>
+          <param name="can_interface_name">can0</param>
+          <param name="auto_start">true</param>
+          <param name="cycle_period_us">1000</param>
+          <param name="target_units_per_rev">10000</param>
+          <param name="slewing_node_id">3</param>
+          <param name="trolley_node_id">2</param>
+          <param name="hoist_node_id">1</param>
+        </hardware>
+        <joint name="slewing_joint">
+          <param name="mechanical_reduction">140.0</param>
+          <command_interface name="position">
+            <param name="min">-3.14</param>
+            <param name="max">3.14</param>
+          </command_interface>
+          <state_interface name="position">
+            <param name="initial_value">${initial_positions['slewing_joint']}</param>
+          </state_interface>
+          <state_interface name="velocity"/>
+        </joint>
+        <joint name="trolley_joint">
+          <param name="mechanical_reduction">10.0</param>
+          <command_interface name="position">
+            <param name="min">-2.0</param>
+            <param name="max">0.5</param>
+          </command_interface>
+          <state_interface name="position">
+            <param name="initial_value">${initial_positions['trolley_joint']}</param>
+          </state_interface>
+          <state_interface name="velocity"/>
+        </joint>
+        <joint name="hook_joint">
+          <param name="mechanical_reduction">40.0</param>
+          <command_interface name="position">
+            <param name="min">0.0</param>
+            <param name="max">2.0</param>
+          </command_interface>
+          <state_interface name="position">
+            <param name="initial_value">${initial_positions['hook_joint']}</param>
+          </state_interface>
+          <state_interface name="velocity"/>
+        </joint>
+      </ros2_control>
+    </xacro:macro>
 </robot>

Commit message: fix: moveit direction wrong

File: crane/tower_crane/urdf/Tower_crane_base.urdf (robot description, URDF)
Before this commit: robot tower_crane, 6 links, 5 joints
Joints:
- joint hook_joint: axis 0 0 1 -> 0 0 -1
- joint slewing_joint: axis 0 0 1 -> 0 0 -1

File: crane/tower_crane/urdf/Tower_crane_base_v2.urdf (robot description, URDF)
Before this commit: robot tower_crane, 6 links, 5 joints
Joints:
- joint hook_joint: axis 0 0 1 -> 0 0 -1
- joint slewing_joint: axis 0 0 1 -> 0 0 -1

File: crane/tower_crane_moveit_config/config/tower_crane.urdf.xacro (robot description, xacro)
@@ -52,5 +52,5 @@
       <parent  link="base_link" />
       <child  link="slewing_Link" />
-      <axis  xyz="0 0 1" />
+      <axis  xyz="0 0 -1" />
       <limit  lower="-3.14"  upper="3.14"  effort="100"  velocity="0" />
     </joint>
@@ -111,5 +111,5 @@
       <parent  link="trolley_Link" />
       <child  link="hook_Link" />
-      <axis  xyz="0 0 1" />
+      <axis  xyz="0 0 -1" />
       <limit  lower="0" upper="2" effort="50" velocity="1.0" />
     </joint>

Commit message: refactor: change movement range

File: crane/tower_crane/urdf/Tower_crane_base.urdf (robot description, URDF)
Before this commit: robot tower_crane, 6 links, 5 joints
Joints:
- joint hook_joint: limit lower=0 upper=2 effort=50 velocity=1.0 -> lower=-2 upper=2 effort=50 velocity=1.0

File: crane/tower_crane_moveit_config/config/tower_crane.urdf.xacro (robot description, xacro)
@@ -112,5 +112,5 @@
       <child  link="hook_Link" />
       <axis  xyz="0 0 -1" />
-      <limit  lower="0" upper="2" effort="50" velocity="1.0" />
+      <limit  lower="-2" upper="2" effort="50" velocity="1.0" />
     </joint>
     <link name="hook_Link">
